Commit message: modify TODO and try to control SO101

File: assets/SO101/so101.urdf (robot description, URDF)
Before this commit: robot so101, 7 links, 8 joints
Links:
- added link base_frame, mass 1e-9
- added link gripper_frame, mass 1e-9
- link base: mass 1e-9 -> 0.147; geometry collision mesh filename=package://assets/base_motor_holder_so101_v1.stl; collision mesh filename=package://assets/base_so101_v2.stl
- link gripper: mass 1e-9 -> 0.087; geometry collision mesh filename=package://assets/sts3215_03a_v1.stl; collision mesh filename=package://assets/wrist_roll_follower_so101_v1.stl
Joints:
- removed joint base_frame
- removed joint gripper_frame
- added joint base_frame_joint: type fixed, parent base, child base_frame, origin xyz=0.020791 0.0157608 0.0324817 rpy=-3.14159 -9.52796e-30 -2.64454e-46, axis 0 0 0
- added joint gripper_frame_joint: type fixed, parent gripper, child gripper_frame, origin xyz=-0.0079 -0.000218121 -0.0981274 rpy=-1.5708 -0 -1.5708, axis 0 0 0
